File: PCB/FRDM-MCXx_Shield/Sensors.kicad_sch (KiCad schematic)
At the start: 8 parts, among them J7 Conn_01x06_Socket, U2 FXLS8974CF

Commit message: Updated PCB and added bill of materials
Parts:
- C7, C9: GPN (none) -> GPC0603104
- C8: GPN (none) -> GPC0603105
- J7: GPN (none) -> GPHA-1X06
Changed lines of the file:
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@@
+      (effects (font (size 1.27 1.27)) hide)
+    )
+    (property "GPN" "GPC0603104" (at 124.46 57.15 0)
       (effects (font (size 1.27 1.27)) hide)
     )
@@
       (effects (font (size 1.27 1.27)) hide)
     )
+    (property "GPN" "GPHA-1X06" (at 76.2 153.67 0)
+      (effects (font (size 1.27 1.27)) hide)
+    )
     (pin "5")
     (pin "3")
@@
       (effects (font (size 1.27 1.27)) hide)
     )
+    (property "GPN" "GPC0603104" (at 46.99 54.61 90)
+      (effects (font (size 1.27 1.27)) hide)
+    )
     (pin "2")
     (pin "1")
@@
       (effects (font (size 1.27 1.27)) hide)
     )
+    (property "GPN" "GPC0603105" (at 113.03 57.15 0)
+      (effects (font (size 1.27 1.27)) hide)
+    )
