File: PCB/FRDM-MCXx_Shield/FRDM-MCXx_Shield.kicad_pcb (KiCad board)
At the start: 4 copper layers, 54.3 x 54.7 mm, 91 parts, among them J1 Conn_02x08_Odd_Even, J2 Conn_02x06_Odd_Even, J3 Conn_02x10_Odd_Even, J4 Conn_02x08_Odd_Even, J5 Conn_01x04_Socket, J6 Conn_01x04_Pin, J7 Conn_01x04_Pin, J8 Conn_01x04_Pin, M1 Motor_Servo, SW1 EC12D1524406, U1 74HC595, U2 M95010-RMN6TP, U3 LM35-D

Commit message: Committed latest changes
Parts:
- removed kibuzzard-65C7C452: G***, kibuzzard-65C7C452
- removed kibuzzard-65C7C5A7: G***, kibuzzard-65C7C5A7
- removed kibuzzard-65C7C5C0: G***, kibuzzard-65C7C5C0
- removed kibuzzard-65C7C5CF: G***, kibuzzard-65C7C5CF
- removed kibuzzard-65C7C73C: G***, kibuzzard-65C7C73C
- removed kibuzzard-65C7C751 (x3): G***, kibuzzard-65C7C751
- removed kibuzzard-65C7C77A (x3): G***, kibuzzard-65C7C77A
- removed kibuzzard-65C7CB3C: G***, kibuzzard-65C7CB3C
- removed kibuzzard-65C7CF02: G***, kibuzzard-65C7CF02
- removed kibuzzard-65C7CF1C: G***, kibuzzard-65C7CF1C
- removed kibuzzard-65D5C7B2: G***, kibuzzard-65D5C7B2
- removed kibuzzard-65D5C7BA (x2): G***, kibuzzard-65D5C7BA
- removed kibuzzard-65D750FF: G***, kibuzzard-65D750FF
- removed kibuzzard-65D9ED05: G***, kibuzzard-65D9ED05
- removed kibuzzard-65D9F158: G***, kibuzzard-65D9F158
- removed kibuzzard-65D9F1EE: G***, kibuzzard-65D9F1EE
- removed kibuzzard-65D9F4C2: G***, kibuzzard-65D9F4C2
- removed kibuzzard-65D9F652: G***, kibuzzard-65D9F652
- removed kibuzzard-65D9F74D: G***, kibuzzard-65D9F74D
- removed kibuzzard-65D9F92F: G***, kibuzzard-65D9F92F
- removed kibuzzard-65D9F962: G***, kibuzzard-65D9F962
- added G***: easteregg, User:easteregg, B.Cu at (168.5, 90.9)
- added H1: MountingHole, MountingHole:MountingHole_2.2mm_M2, F.Cu at (129.3, 79.8)
- added H2: MountingHole, MountingHole:MountingHole_2.2mm_M2, F.Cu at (129.3, 102.1)
- added kibuzzard-662EB4EE: G***, kibuzzard-662EB4EE, F.Cu at (136.6, 72.0)
- added kibuzzard-662EB530: G***, kibuzzard-662EB530, F.Cu at (140.6, 77.2)
- added kibuzzard-662EB540: G***, kibuzzard-662EB540, F.Cu at (135.4, 77.2)
- added kibuzzard-662EB54B: G***, kibuzzard-662EB54B, F.Cu at (138.1, 77.2)
- added kibuzzard-662EB5D9: G***, kibuzzard-662EB5D9, F.Cu at (133.0, 77.2)
- added kibuzzard-662EB6D3: G***, kibuzzard-662EB6D3, F.Cu at (132.4, 87.3)
- added kibuzzard-662EB6E1: G***, kibuzzard-662EB6E1, F.Cu at (132.3, 89.8)
- added kibuzzard-662EB6F1: G***, kibuzzard-662EB6F1, F.Cu at (132.6, 92.3)
- added kibuzzard-662EB702: G***, kibuzzard-662EB702, F.Cu at (132.4, 94.9)
- added kibuzzard-662EB7B6: G***, kibuzzard-662EB7B6, F.Cu at (135.3, 91.0)
- added kibuzzard-662EB81C: G***, kibuzzard-662EB81C, B.Cu at (136.5, 90.4)
- added kibuzzard-662EB828: G***, kibuzzard-662EB828, B.Cu at (136.8, 92.3)
- added kibuzzard-662EB833: G***, kibuzzard-662EB833, B.Cu at (136.8, 94.3)
- added kibuzzard-662EB85A: G***, kibuzzard-662EB85A, B.Cu at (131.5, 92.1)
- added kibuzzard-662EB907: G***, kibuzzard-662EB907, F.Cu at (168.5, 72.0)
- added kibuzzard-662EB9E9: G***, kibuzzard-662EB9E9, F.Cu at (160.6, 114.2)
- added kibuzzard-662EBA34: G***, kibuzzard-662EBA34, F.Cu at (151.3, 74.2)
- added kibuzzard-662EBB86: G***, kibuzzard-662EBB86, F.Cu at (153.2, 111.0)
- added kibuzzard-662EC8A0: G***, kibuzzard-662EC8A0, F.Cu at (142.6, 101.1)
- added kibuzzard-662EC8AF: G***, kibuzzard-662EC8AF, F.Cu at (146.0, 99.5)
- added kibuzzard-662ECA3B: G***, kibuzzard-662ECA3B, F.Cu at (139.0, 103.4)
- ?, C9, D12, RN1: moved to B.Cu
- moved SSD1306 68.7 mm to (120.9, 157.3), turned to 0 degrees
- moved D12 15.5 mm to (168.5, 90.9), turned to 180 degrees
- moved ? 13.3 mm to (145.4, 96.7)
- moved D10 12.1 mm to (151.8, 80.0)
- moved D11 9.77 mm to (139.7, 84.4), turned to 180 degrees
- moved D1 8.47 mm to (157.5, 90.9), turned to 180 degrees
- moved D2 8.46 mm to (160.7, 83.2), turned to 135 degrees
- moved D8 8.45 mm to (160.7, 98.7), turned to -135 degrees
- moved D3 8.42 mm to (168.5, 79.9), turned to 90 degrees
- moved D7 8.42 mm to (168.5, 101.9), turned to -90 degrees
- moved D4 8.39 mm to (176.3, 83.2), turned to 45 degrees
- moved D6 8.38 mm to (176.3, 98.7), turned to -45 degrees
- moved D5 8.37 mm to (179.5, 90.9), turned to 0 degrees
- moved C9 5.80 mm to (146.9, 72.7), turned to 180 degrees
- moved TP2 4.02 mm to (157.2, 101.0)
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Connections:
- RN2 pad 1: Net-(D5-A) -> Net-(D4-A)
- RN2 pad 2: Net-(D6-A) -> Net-(D3-A)
- RN2 pad 3: Net-(D7-A) -> Net-(D2-A)
- RN2 pad 4: Net-(D8-A) -> Net-(D1-A)
- RN3 pad 1: Net-(D4-A) -> Net-(D5-A)
- RN3 pad 2: Net-(D3-A) -> Net-(D6-A)
- RN3 pad 3: Net-(D2-A) -> Net-(D7-A)
- RN3 pad 4: Net-(D1-A) -> Net-(D8-A)
Routing:
- net +3.3V: track 37.0 -> 287.0 mm, vias 0 -> 13
- net /~{SHIFTREG_CS}: track 0.00 -> 105.0 mm, vias 0 -> 2
- net /SPI_MISO: track 13.2 -> 108.6 mm, vias 0 -> 2
- net /~{SHIFTREG_RST}: track 0.00 -> 94.3 mm, vias 0 -> 2
- net Net-(D2-A): track 0.00 -> 88.2 mm, vias 0 -> 2
- net /SPI_CLK: track 7.81 -> 93.3 mm, vias 0 -> 3
- net /~{EEPROM_CS}: track 0.00 -> 81.5 mm, vias 0 -> 4
- net Net-(D1-A): track 0.00 -> 75.8 mm, vias 0 -> 3
- net /SPI_MOSI: track 7.53 -> 82.0 mm, vias 0 -> 2
- net /SERVO_PWM: track 3.53 -> 77.3 mm
- net Net-(D8-A): track 0.00 -> 49.9 mm, vias 0 -> 2
- net /WRITE_PROT: track 4.17 -> 53.9 mm, vias 0 -> 2
- net +5V: track 7.32 -> 52.6 mm, vias 0 -> 1
- net Net-(D7-A): track 0.00 -> 36.6 mm, vias 0 -> 2
- net Net-(D6-A): track 0.00 -> 27.8 mm, vias 0 -> 2
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