File: PCB/FRDM-MCXx_Shield_V3.0/FRDM-MCXx_Shield_V3.0.kicad_sch (KiCad schematic)
At the start: 10 parts, among them J1 Conn_02x08_Odd_Even, J2 Conn_02x06_Odd_Even, J3 Conn_02x10_Odd_Even, J4 Conn_02x08_Odd_Even

Commit message: Added R7
Changed lines of the file:
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@@
 	(title_block
 		(title "Main")
-		(date "2024-06-17")
+		(date "2024-06-19")
 		(rev "V3.0")
 		(company "HAN")
@@
 		)
 	)
-	(text_box "Changes V3.0:\n - Removed capacitor at encoder input.\n - Removed MISO connection with shiftregister.\n \n - Changed 3.3V to 5V at the LM35 power input.  \n - Changed P3_12 to P3_10.\n"
+	(text_box "Changes V3.0:\n - Removed capacitor at encoder input.\n - Removed MISO connection with shiftregister.\n \n - Changed 3.3V to 5V at the LM35 power input.  \n - Changed P3_12 to P3_10.\n\n - Added termination resistor at neopixel data line."
 		(exclude_from_sim no)
 		(at 16.51 161.29 0)
@@
 		)
 		(instances
-			(project "FRDM-MCXx_Shield"
+			(project "FRDM-MCXx_Shield_V3.0"
 				(path "/bffc27af-f9e0-4cc8-b5dc-88d2faf26a17"
 					(reference "J4")
@@
 		)
 		(instances
-			(project "FRDM-MCXx_Shield"
+			(project "FRDM-MCXx_Shield_V3.0"
 				(path "/bffc27af-f9e0-4cc8-b5dc-88d2faf26a17"
 					(reference "RN1")
@@
 		)
 		(instances
-			(project "FRDM-MCXx_Shield"
+			(project "FRDM-MCXx_Shield_V3.0"
 				(path "/bffc27af-f9e0-4cc8-b5dc-88d2faf26a17"
 					(reference "#PWR05")
@@
 		)
 		(instances
-			(project "FRDM-MCXx_Shield"
+			(project "FRDM-MCXx_Shield_V3.0"
 				(path "/bffc27af-f9e0-4cc8-b5dc-88d2faf26a17"
 					(reference "#PWR02")
@@
 		)
 		(instances
-			(project "FRDM-MCXx_Shield"
+			(project "FRDM-MCXx_Shield_V3.0"
 				(path "/bffc27af-f9e0-4cc8-b5dc-88d2faf26a17"
 					(reference "REF1")
@@
 		)
 		(instances
-			(project "FRDM-MCXx_Shield"
+			(project "FRDM-MCXx_Shield_V3.0"
 				(path "/bffc27af-f9e0-4cc8-b5dc-88d2faf26a17"
 					(reference "H2")
@@
 		)
 		(instances
-			(project "FRDM-MCXx_Shield"
+			(project "FRDM-MCXx_Shield_V3.0"
 				(path "/bffc27af-f9e0-4cc8-b5dc-88d2faf26a17"
 					(reference "H1")
@@
 		)
 		(instances
-			(project "FRDM-MCXx_Shield"
+			(project "FRDM-MCXx_Shield_V3.0"
 				(path "/bffc27af-f9e0-4cc8-b5dc-88d2faf26a17"
 					(reference "#PWR01")
@@
 		)
 		(instances
-			(project "FRDM-MCXx_Shield"
+			(project "FRDM-MCXx_Shield_V3.0"
 				(path "/bffc27af-f9e0-4cc8-b5dc-88d2faf26a17"
 					(reference "J1")
@@
 		)
 		(instances
-			(project "FRDM-MCXx_Shield"
+			(project "FRDM-MCXx_Shield_V3.0"
 				(path "/bffc27af-f9e0-4cc8-b5dc-88d2faf26a17"
 					(reference "RN1")
@@
 		)
 		(instances
-			(project "FRDM-MCXx_Shield"
+			(project "FRDM-MCXx_Shield_V3.0"
 				(path "/bffc27af-f9e0-4cc8-b5dc-88d2faf26a17"
 					(reference "#PWR03")
@@
 		)
 		(instances
-			(project "FRDM-MCXx_Shield"
+			(project "FRDM-MCXx_Shield_V3.0"
 				(path "/bffc27af-f9e0-4cc8-b5dc-88d2faf26a17"
 					(reference "REF2")
@@
 		)
 		(instances
-			(project "FRDM-MCXx_Shield"
+			(project "FRDM-MCXx_Shield_V3.0"
 				(path "/bffc27af-f9e0-4cc8-b5dc-88d2faf26a17"
 					(reference "J2")
@@
 		)
 		(instances
-			(project "FRDM-MCXx_Shield"
+			(project "FRDM-MCXx_Shield_V3.0"
 				(path "/bffc27af-f9e0-4cc8-b5dc-88d2faf26a17"
 					(reference "J3")
@@
 		)
 		(instances
-			(project "FRDM-MCXx_Shield"
+			(project "FRDM-MCXx_Shield_V3.0"
 				(path "/bffc27af-f9e0-4cc8-b5dc-88d2faf26a17"
 					(reference "#PWR04")
@@
 		)
 		(instances
-			(project "FRDM-MCXx_Shield"
+			(project "FRDM-MCXx_Shield_V3.0"
 				(path "/bffc27af-f9e0-4cc8-b5dc-88d2faf26a17"
 					(reference "REF3")
@@
 		)
 		(instances
-			(project "FRDM-MCXx_Shield"
+			(project "FRDM-MCXx_Shield_V3.0"
 				(path "/bffc27af-f9e0-4cc8-b5dc-88d2faf26a17"
 					(page "3")
@@
 		)
 		(instances
-			(project "FRDM-MCXx_Shield"
+			(project "FRDM-MCXx_Shield_V3.0"
 				(path "/bffc27af-f9e0-4cc8-b5dc-88d2faf26a17"
 					(page "2")
@@
 		)
 		(instances
-			(project "FRDM-MCXx_Shield"
+			(project "FRDM-MCXx_Shield_V3.0"
 				(path "/bffc27af-f9e0-4cc8-b5dc-88d2faf26a17"
 					(page "4")
