File: PCB/FRDM-MCXx_Shield_V3.0/HMI.kicad_sch (KiCad schematic)
At the start: 25 parts, among them J5 Conn_01x04_Socket, SW1 EC12D1524406, U1 74HC595

Commit message: Updated assembly
Parts:
- R1, R3, R4: now fitted
Changed lines of the file:
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@@
 	(title_block
 		(title "HMI")
-		(date "2024-06-17")
+		(date "2024-06-20")
 		(rev "V3.0")
 		(company "HAN")
@@
 		(in_bom yes)
 		(on_board yes)
-		(dnp yes)
+		(dnp no)
 		(fields_autoplaced yes)
 		(property "Reference" "R4"
@@
 		(in_bom yes)
 		(on_board yes)
-		(dnp yes)
+		(dnp no)
 		(fields_autoplaced yes)
 		(property "Reference" "R1"
@@
 		(in_bom yes)
 		(on_board yes)
-		(dnp yes)
+		(dnp no)
 		(fields_autoplaced yes)
 		(property "Reference" "R3"
